Commit message: Add the Robosense Helios 32 LiDAR

File: urdf/husky.urdf.xacro (robot description, xacro)
@@ -26,4 +26,22 @@
   <xacro:arg name="imu_rpy"     default="$(optenv HUSKY_IMU_RPY 0 -1.5708 3.1416)"/>
   <xacro:arg name="imu_parent"  default="$(optenv HUSKY_IMU_PARENT base_link)"/>
+  <!-- Robosense Helios 32 3D LIDAR -->
+  <xacro:include filename="$(find husky_slam)/urdf/robosense.urdf.xacro"/>
+  <xacro:RS-32
+    parent="top_plate_link"
+    name="helios32"
+    topic="/helios32/points"
+    hz="10"
+    lasers="32"
+    samples="1200"
+    collision_range="0.4"
+    min_range="0.4"
+    max_range="150.0"
+    noise="0.008"
+    min_angle="-3.14159"
+    max_angle="3.14159"
+    gpu="true">
+    <origin xyz="0 0 0" rpy="0 0 0"/>
+  </xacro:RS-32>
   <!-- LMS1XX Laser Primary and Secondary -->
   <xacro:arg name="laser_enabled"           default="$(optenv HUSKY_LMS1XX_ENABLED 0)" />

Commit message: Add the platform for the LiDAR

File: urdf/husky.urdf.xacro (robot description, xacro)
@@ -29,5 +29,5 @@
   <xacro:include filename="$(find husky_slam)/urdf/robosense.urdf.xacro"/>
   <xacro:RS-32
-    parent="top_plate_link"
+    parent="lidar_platform_link"
     name="helios32"
     topic="/helios32/points"
@@ -42,5 +42,5 @@
     max_angle="3.14159"
     gpu="true">
-    <origin xyz="0 0 0" rpy="0 0 0"/>
+    <origin xyz="0 0 0.07" rpy="0 0 0"/>
   </xacro:RS-32>
   <!-- LMS1XX Laser Primary and Secondary -->
@@ -196,4 +196,33 @@
     <child link="inertial_link" />
   </joint>
+  <!-- Robosense platform -->
+  <link name="lidar_platform_link">
+    <visual>
+      <origin xyz="0 0 0.025" rpy="0 0 0"/>
+      <geometry>
+        <box size="0.15 0.15 0.08"/>
+      </geometry>
+      <material name="platform_gray">
+        <color rgba="0.5 0.5 0.5 1.0"/>
+      </material>
+    </visual>
+    <collision>
+      <origin xyz="0 0 00.025" rpy="0 0 0"/>
+      <geometry>
+        <box size="0.15 0.15 0.08"/>
+      </geometry>
+    </collision>
+    <inertial>
+      <mass value="0.1"/>
+      <inertia ixx="0.001" ixy="0.0" ixz="0.0"
+              iyy="0.001" iyz="0.0"
+              izz="0.001"/>
+    </inertial>
+  </link>
+  <joint name="lidar_platform_joint" type="fixed">
+    <parent link="top_plate_link"/>
+    <child link="lidar_platform_link"/>
+    <origin xyz="0 0 0.025" rpy="0 0 0"/>
+  </joint>
   <!-- Husky wheel macros -->
   <xacro:husky_wheel wheel_prefix="front_left">

Commit message: Remove the lidar platform and add the sensor arch

File: urdf/husky.urdf.xacro (robot description, xacro)
@@ -29,5 +29,5 @@
   <xacro:include filename="$(find husky_slam)/urdf/robosense.urdf.xacro"/>
   <xacro:RS-32
-    parent="lidar_platform_link"
+    parent="top_plate_link"
     name="helios32"
     topic="/helios32/points"
@@ -42,5 +42,5 @@
     max_angle="3.14159"
     gpu="true">
-    <origin xyz="0 0 0.07" rpy="0 0 0"/>
+    <origin xyz="0 0 0.025" rpy="0 0 0"/>
   </xacro:RS-32>
   <!-- LMS1XX Laser Primary and Secondary -->
@@ -92,5 +92,5 @@
   <xacro:arg name="realsense_topic"               default="$(optenv HUSKY_REALSENSE_TOPIC realsense)" />
   <xacro:arg name="realsense_prefix"              default="$(optenv HUSKY_REALSENSE_PREFIX camera)" />
-  <xacro:arg name="realsense_parent"              default="$(optenv HUSKY_REALSENSE_PARENT top_plate_link)" />
+  <xacro:arg name="realsense_parent"              default="$(optenv HUSKY_REALSENSE_PARENT sensor_arch_mount_link)" />
   <xacro:arg name="realsense_xyz"                 default="$(optenv HUSKY_REALSENSE_XYZ 0 0 0)" />
   <xacro:arg name="realsense_rpy"                 default="$(optenv HUSKY_REALSENSE_RPY 0 0 0)" />
@@ -196,10 +196,10 @@
     <child link="inertial_link" />
   </joint>
-  <!-- Robosense platform -->
+  <!-- Robosense platform
   <link name="lidar_platform_link">
     <visual>
-      <origin xyz="0 0 0.025" rpy="0 0 0"/>
+      <origin xyz="0.05 0.05 0.025" rpy="0 0 0"/>
       <geometry>
-        <box size="0.15 0.15 0.08"/>
+        <box size="0.15 0.15 0.05"/>
       </geometry>
       <material name="platform_gray">
@@ -208,7 +208,7 @@
     </visual>
     <collision>
-      <origin xyz="0 0 00.025" rpy="0 0 0"/>
+      <origin xyz="0.05 0.05 0.025" rpy="0 0 0"/>
       <geometry>
-        <box size="0.15 0.15 0.08"/>
+        <box size="0.15 0.15 0.05"/>
       </geometry>
     </collision>
@@ -223,6 +223,7 @@
     <parent link="top_plate_link"/>
     <child link="lidar_platform_link"/>
-    <origin xyz="0 0 0.025" rpy="0 0 0"/>
+    <origin xyz="0.05 0.05 0.02" rpy="0 0 0"/>
   </joint>
+  -->
   <!-- Husky wheel macros -->
   <xacro:husky_wheel wheel_prefix="front_left">
